File: Artemis Payload Computer/BAROMETER.sch (KiCad schematic (older format))
At the start: 0 parts

Commit message: Added BMP280 and IMU to the schematic
Parts:
- added U?: BMP280, symbol Artemis_Footprints:BMP280
Changed lines of the file:
@@
 $Descr A4 11693 8268
 encoding utf-8
-Sheet 1 4
+Sheet 3 4
 Title ""
 Date ""
@@
 Comment4 ""
 $EndDescr
+$Comp
+L Artemis_Footprints:BMP280 U?
+U 1 1 603A8ECA
+P 6100 3650
+F 0 "U?" H 6125 4015 50  0000 C CNN
+F 1 "BMP280" H 6125 3924 50  0000 C CNN
+F 2 "" H 6100 4150 50  0001 C CNN
+F 3 "" H 6100 4150 50  0001 C CNN
+	1    6100 3650
+	1    0    0    -1
+$EndComp
 $EndSCHEMATC
