File: Artemis Payload Computer/IMU.sch (KiCad schematic (older format))
At the start: 0 parts

Commit message: Added BMP280 and IMU to the schematic
Parts:
- added U?: FXOS8700+FXAS21002, symbol Artemis_Footprints:FXOS8700+FXAS21002
Changed lines of the file:
@@
 $Descr A4 11693 8268
 encoding utf-8
-Sheet 1 4
+Sheet 4 4
 Title ""
 Date ""
@@
 Comment4 ""
 $EndDescr
+$Comp
+L Artemis_Footprints:FXOS8700+FXAS21002 U?
+U 1 1 603A9652
+P 6250 3450
+F 0 "U?" H 6275 3965 50  0000 C CNN
+F 1 "FXOS8700+FXAS21002" H 6275 3874 50  0000 C CNN
+F 2 "" H 6250 3450 50  0001 C CNN
+F 3 "" H 6250 3450 50  0001 C CNN
+	1    6250 3450
+	1    0    0    -1
+$EndComp
 $EndSCHEMATC
