File: Artemis Payload Computer/Artemis Payload Computer.sch (KiCad schematic (older format))
At the start: 0 parts

Commit message: Added Voltage Regulator
Changed lines of the file:
@@
 $Descr A4 11693 8268
 encoding utf-8
-Sheet 1 4
+Sheet 1 5
 Title ""
 Date ""
@@
 F1 "IMU.sch" 50
 $EndSheet
+$Sheet
+S 1750 5300 1350 950
+U 603A9972
+F0 "Power Supply" 50
+F1 "Power Supply.sch" 50
+$EndSheet
 $EndSCHEMATC
