File: Artemis Payload Computer/WS STRAIN GAUGE.sch (KiCad schematic (older format))
At the start: 5 parts, among them J1 Screw_Terminal_01x02, J2 Screw_Terminal_01x02, U1 HX711

Commit message: Updated Footprints
Parts:
- J1, J2: footprint (none) -> TerminalBlock_TE-Connectivity:TerminalBlock_TE_282834-2_1x02_P2.54mm_Horizontal
- R1, R2: footprint (none) -> Resistor_SMD:R_0603_1608Metric_Pad0.98x0.95mm_HandSolder
Changed lines of the file:
@@
 F 0 "R2" H 5330 3050 50  0000 C CNN
 F 1 "R_US" H 5370 2960 50  0000 C CNN
-F 2 "" V 5270 3020 50  0001 C CNN
+F 2 "Resistor_SMD:R_0603_1608Metric_Pad0.98x0.95mm_HandSolder" V 5270 3020 50  0001 C CNN
 F 3 "~" H 5230 3030 50  0001 C CNN
 	1    5230 3030
@@
 F 0 "R1" H 5030 3000 50  0000 R CNN
 F 1 "R_US" H 5130 3080 50  0000 R CNN
-F 2 "" V 4930 3020 50  0001 C CNN
+F 2 "Resistor_SMD:R_0603_1608Metric_Pad0.98x0.95mm_HandSolder" V 4930 3020 50  0001 C CNN
 F 3 "~" H 4890 3030 50  0001 C CNN
 	1    4890 3030
@@
 F 0 "J1" H 4810 2630 50  0000 C CNN
 F 1 "Screw_Terminal_01x02" H 5180 2700 50  0000 C CNN
-F 2 "" H 4690 2670 50  0001 C CNN
+F 2 "TerminalBlock_TE-Connectivity:TerminalBlock_TE_282834-2_1x02_P2.54mm_Horizontal" H 4690 2670 50  0001 C CNN
 F 3 "~" H 4690 2670 50  0001 C CNN
 	1    4690 2670
@@
 F 0 "J2" H 5510 2562 50  0000 L CNN
 F 1 "Screw_Terminal_01x02" H 5510 2471 50  0000 L CNN
-F 2 "" H 5430 2570 50  0001 C CNN
+F 2 "TerminalBlock_TE-Connectivity:TerminalBlock_TE_282834-2_1x02_P2.54mm_Horizontal" H 5430 2570 50  0001 C CNN
 F 3 "~" H 5430 2570 50  0001 C CNN
 	1    5430 2570

Commit message: Fixed Strain Gauge Footprint
Parts:
- U1: footprint .pretty:HX711 -> Artemis Payload Computer:HX711
Changed lines of the file:
@@
 F 0 "U1" H 6930 3210 50  0001 L BNN
 F 1 "HX711" H 6930 3210 50  0001 L BNN
-F 2 ".pretty:HX711" H 6930 3210 50  0001 L BNN
+F 2 "Artemis Payload Computer:HX711" H 6930 3210 50  0001 L BNN
 F 3 "" H 6930 3210 50  0001 L BNN
 	1    6930 3210
