File: Artemis Payload Computer/BMP280.sch (KiCad schematic (older format))
At the start: 1 part, among them U501 BMP280

Commit message: ready for testing...
Connections:
- net +5V: now reaches U501.1 (VIN)
- net GND: now reaches U501.3 (GND)
- net SCL0: now reaches U501.4 (SCK)
- net SDA0: now reaches U501.6 (SDI)
Changed lines of the file:
@@
 	1    0    0    -1
 $EndComp
+$Comp
+L power:+5V #PWR0111
+U 1 1 60406C8A
+P 5250 3500
+F 0 "#PWR0111" H 5250 3350 50  0001 C CNN
+F 1 "+5V" V 5265 3628 50  0000 L CNN
+F 2 "" H 5250 3500 50  0001 C CNN
+F 3 "" H 5250 3500 50  0001 C CNN
+	1    5250 3500
+	0    -1   -1   0
+$EndComp
+$Comp
+L power:GND #PWR0112
+U 1 1 60406EDA
+P 5250 3700
+F 0 "#PWR0112" H 5250 3450 50  0001 C CNN
+F 1 "GND" V 5255 3572 50  0000 R CNN
+F 2 "" H 5250 3700 50  0001 C CNN
+F 3 "" H 5250 3700 50  0001 C CNN
+	1    5250 3700
+	0    1    1    0
+$EndComp
+Text HLabel 6400 3500 2    50   Input ~ 0
+SCL0
+Text HLabel 6400 3700 2    50   Input ~ 0
+SDA0
+Wire Wire Line
+	6200 3700 6400 3700
+Wire Wire Line
+	6200 3500 6400 3500
+Wire Wire Line
+	5450 3500 5250 3500
+Wire Wire Line
+	5250 3700 5450 3700
 $EndSCHEMATC
